File: mk2.brd (EAGLE design)
At the start: 31.2 x 31.6 mm, 20 parts, among them IC1 78L05F, Q1 16MHz, U1 ATMEGA328P-AU

Commit message: Some cleanup.
Parts:
- R2, R3, R4: value (none) -> 470R
- moved S1 15.7 mm to (30.6, 5.33)
- moved S2 15.7 mm to (30.6, 21.1)
Connections:
- net GND: now also S2.2; no longer S1.2
- net N$15: now also S2.1; no longer S1.1
- net PWR: now also S1.1; no longer S2.1
- net VCC: now also S1.2; no longer S2.2
Changed lines of the file:
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@@
 <?xml version="1.0" encoding="utf-8"?>
 <!DOCTYPE eagle SYSTEM "eagle.dtd">
-<eagle version="8.4.0">
+<eagle version="8.3.1">
 <drawing>
 <settings>
@@
 <dimension x1="0.889" y1="33.645" x2="0.889" y2="2.032" x3="-2.54" y3="17.8385" textsize="1.778" layer="49"/>
 <dimension x1="0.889" y1="2.032" x2="32.131" y2="2.032" x3="16.51" y3="-2.794" textsize="1.778" layer="47"/>
-<text x="16.51" y="31.242" size="0.8128" layer="21" font="fixed" align="center">dtctr
+<text x="16.51" y="31.75" size="0.8128" layer="21" font="fixed" align="center">dtctr
 uberbadassequipment.com</text>
 <text x="2.032" y="31.847365625" size="1.778" layer="21" align="center">-</text>
@@
 <param name="dpMaxLengthDifference" value="10mm"/>
 <param name="dpGapFactor" value="2.5"/>
+<param name="checkGrid" value="0"/>
+<param name="checkAngle" value="0"/>
 <param name="checkFont" value="1"/>
 <param name="checkRestrict" value="1"/>
-<param name="checkStop" value="0"/>
 <param name="useDiameter" value="13"/>
 <param name="maxErrors" value="50"/>
@@
 <attribute name="VALUE" x="28.06696875" y="16.51" size="1.27" layer="27" rot="R270"/>
 </element>
-<element name="R2" library="resistor" package="M1206" value="" x="26.2524875" y="15.24" smashed="yes" rot="R90">
+<element name="R2" library="resistor" package="M1206" value="470R" x="26.2524875" y="15.24" smashed="yes" rot="R90">
 <attribute name="NAME" x="24.9824875" y="13.97" size="1.27" layer="25" rot="R90"/>
 <attribute name="VALUE" x="28.7924875" y="13.97" size="1.27" layer="27" rot="R90"/>
 </element>
-<element name="R3" library="resistor" package="M1206" value="" x="21.89800625" y="15.24" smashed="yes" rot="R90">
+<element name="R3" library="resistor" package="M1206" value="470R" x="21.89800625" y="15.24" smashed="yes" rot="R90">
 <attribute name="NAME" x="20.62800625" y="13.97" size="1.27" layer="25" rot="R90"/>
 <attribute name="VALUE" x="24.43800625" y="13.97" size="1.27" layer="27" rot="R90"/>
 </element>
-<element name="R4" library="resistor" package="M1206" value="" x="11.193525" y="15.24" smashed="yes" rot="R90">
+<element name="R4" library="resistor" package="M1206" value="470R" x="11.193525" y="15.24" smashed="yes" rot="R90">
 <attribute name="NAME" x="9.923525" y="13.97" size="1.27" layer="25" rot="R90"/>
 <attribute name="VALUE" x="13.733525" y="13.97" size="1.27" layer="27" rot="R90"/>
@@
 <attribute name="NAME" x="24.13" y="5.08" size="1.27" layer="25"/>
 </element>
-<element name="S2" library="SparkFun-Electromechanical" package="TACTILE_SWITCH-SMD-RIGHT-ANGLE" value="SWITCH-MOMENTARY-2TACTILE-SWITCH-SMD-RIGHT-ANGLE" x="30.607" y="5.334" rot="R90">
+<element name="S1" library="SparkFun-Electromechanical" package="TACTILE_SWITCH-SMD-RIGHT-ANGLE" value="SWITCH-MOMENTARY-2TACTILE-SWITCH-SMD-RIGHT-ANGLE" x="30.607" y="5.334" rot="R90">
 <attribute name="PROD_ID" value="COMP-12265" x="30.607" y="5.334" size="1.778" layer="27" rot="R90" display="off"/>
 </element>
@@
 </element>
 <element name="X1" library="adafruit" package="HDF15V" value="" x="16.51" y="26.67" rot="MR180"/>
-<element name="S1" library="SparkFun-Electromechanical" package="TACTILE_SWITCH-SMD-RIGHT-ANGLE" value="SWITCH-MOMENTARY-2TACTILE-SWITCH-SMD-RIGHT-ANGLE" x="30.607" y="21.082" rot="R90">
+<element name="S2" library="SparkFun-Electromechanical" package="TACTILE_SWITCH-SMD-RIGHT-ANGLE" value="SWITCH-MOMENTARY-2TACTILE-SWITCH-SMD-RIGHT-ANGLE" x="30.607" y="21.082" rot="R90">
 <attribute name="PROD_ID" value="COMP-12265" x="30.607" y="21.082" size="1.778" layer="27" rot="R90" display="off"/>
 </element>
@@
 <vertex x="0" y="34.29"/>
 </polygon>
-<contactref element="S1" pad="2"/>
+<contactref element="S2" pad="2"/>
 <contactref element="LED1" pad="C"/>
 <contactref element="LED2" pad="C"/>
@@
 </signal>
 <signal name="VCC">
-<contactref element="S2" pad="2"/>
+<contactref element="S1" pad="2"/>
 <contactref element="U1" pad="4"/>
 <contactref element="U1" pad="6"/>
@@
 </signal>
 <signal name="PWR">
-<contactref element="S2" pad="1"/>
+<contactref element="S1" pad="1"/>
 <contactref element="U$1" pad="+$2"/>
-<contactref element="U$1" pad="+$1"/>
 <contactref element="IC1" pad="1"/>
 <wire x1="28.7528" y1="4.9784" x2="30.5816" y2="3.1496" width="0.254" layer="1"/>
@@
 <wire x1="3.8608" y1="11.8872" x2="5.2832" y2="13.3096" width="0.254" layer="16"/>
 <wire x1="3.4544" y1="22.4536" x2="3.48" y2="22.454" width="0.254" layer="1"/>
-<wire x1="3.8608" y1="11.8872" x2="3.81" y2="11.811" width="0.254" layer="16"/>
 <wire x1="29.2608" y1="16.3576" x2="29.2608" y2="11.8872" width="0.254" layer="16"/>
 <wire x1="29.7688" y1="16.8656" x2="29.2608" y2="16.3576" width="0.254" layer="16"/>
@@
 <via x="8.7376" y="30.1752" extent="1-16" drill="0.3302"/>
 <via x="7.8232" y="29.2608" extent="1-16" drill="0.3302"/>
+<contactref element="U$1" pad="+$1"/>
+<wire x1="3.81" y1="11.811" x2="3.8608" y2="11.8872" width="0" layer="19" extent="16-16"/>
 </signal>
 <signal name="N$8">
@@
 </signal>
 <signal name="N$15">
-<contactref element="S1" pad="1"/>
+<contactref element="S2" pad="1"/>
 <contactref element="U1" pad="16"/>
 <wire x1="21.4376" y1="8.8392" x2="21.4376" y2="7.7216" width="0.254" layer="1"/>
