File: mk2.sch (EAGLE design)
At the start: 20 parts, among them IC1 78L05F, Q1 16MHz, U1 ATMEGA328P-AU

Commit message: Some cleanup.
Parts:
- R2, R3, R4: value (none) -> 470R
Connections:
- net GND: now also S2.2; no longer S1.2
- net N$15: now also S2.1; no longer S1.1
- net PWR: now also S1.1; no longer S2.1
- net VCC: now also S1.2; no longer S2.2
Other:
- note removed: "Note: R2-4 @3V: 240R @5V 470R"
- moved on the sheet: JP1, R1, R4, R5, S1, S2, U$1

Commit message: Schematics cleanup. Less aaaaaaah.
Other:
- moved on the sheet: C1, C2, LED1, LED2, Q1, R8, S2
